Commit message: Update classes, Create initial_arm_pose

File: paquetes_simulacion/rb1_base_description/robots/robot.urdf (robot description, URDF)
Before this commit: robot rb1_base, 41 links, 40 joints
Joints:
- joint rb1_left_arm_elbow_joint: limit lower=-3.141592653589793 upper=3.141592653589793 effort=150.0 velocity=3.15 -> lower=-6.283185307179586 upper=6.283185307179586 effort=150.0 velocity=3.15
- joint rb1_left_arm_shoulder_lift_joint: limit lower=-3.141592653589793 upper=3.141592653589793 effort=330.0 velocity=2.16 -> lower=-6.283185307179586 upper=6.283185307179586 effort=330.0 velocity=2.16
- joint rb1_left_arm_shoulder_pan_joint: limit lower=-3.141592653589793 upper=3.141592653589793 effort=330.0 velocity=2.16 -> lower=-6.283185307179586 upper=6.283185307179586 effort=330.0 velocity=2.16
- joint rb1_left_arm_wrist_1_joint: limit lower=-3.141592653589793 upper=3.141592653589793 effort=54.0 velocity=3.2 -> lower=-6.283185307179586 upper=6.283185307179586 effort=54.0 velocity=3.2
- joint rb1_left_arm_wrist_2_joint: limit lower=-3.141592653589793 upper=3.141592653589793 effort=54.0 velocity=3.2 -> lower=-6.283185307179586 upper=6.283185307179586 effort=54.0 velocity=3.2
- joint rb1_left_arm_wrist_3_joint: limit lower=-3.141592653589793 upper=3.141592653589793 effort=54.0 velocity=3.2 -> lower=-6.283185307179586 upper=6.283185307179586 effort=54.0 velocity=3.2
- joint rb1_right_arm_elbow_joint: limit lower=-3.141592653589793 upper=3.141592653589793 effort=150.0 velocity=3.15 -> lower=-6.283185307179586 upper=6.283185307179586 effort=150.0 velocity=3.15
- joint rb1_right_arm_shoulder_lift_joint: limit lower=-3.141592653589793 upper=3.141592653589793 effort=330.0 velocity=2.16 -> lower=-6.283185307179586 upper=6.283185307179586 effort=330.0 velocity=2.16
- joint rb1_right_arm_shoulder_pan_joint: limit lower=-3.141592653589793 upper=3.141592653589793 effort=330.0 velocity=2.16 -> lower=-6.283185307179586 upper=6.283185307179586 effort=330.0 velocity=2.16
- joint rb1_right_arm_wrist_1_joint: limit lower=-3.141592653589793 upper=3.141592653589793 effort=54.0 velocity=3.2 -> lower=-6.283185307179586 upper=6.283185307179586 effort=54.0 velocity=3.2
- joint rb1_right_arm_wrist_2_joint: limit lower=-3.141592653589793 upper=3.141592653589793 effort=54.0 velocity=3.2 -> lower=-6.283185307179586 upper=6.283185307179586 effort=54.0 velocity=3.2
- joint rb1_right_arm_wrist_3_joint: limit lower=-3.141592653589793 upper=3.141592653589793 effort=54.0 velocity=3.2 -> lower=-6.283185307179586 upper=6.283185307179586 effort=54.0 velocity=3.2
