Commit message: Adam_sim without pybullet examples

File: paquetes_simulacion/inspire_hands/inspire_hand_l/urdf/inspire_hand_l.urdf (robot description, URDF)
Before this commit: robot inspire_hand_l, 14 links, 13 joints
Links:
- removed link world
Joints:
- removed joint fixed
- joint L_index_MCP_joint: origin xyz=-0.096414 -0.24897 -0.24007 rpy=-1.3208 -0.034907 3.1416 -> xyz=0.018414 -0.00017 0.13704 rpy=-4.462392654 0.034907 0
- joint L_middle_MCP_joint: origin xyz=-0.077068 -0.24897 -0.24016 rpy=-1.3208 0 3.1416 -> xyz=-0.000932 -0.00017 0.13713 rpy=-4.462392654 0 0
- joint L_pinky_MCP_joint: origin xyz=-0.033256 -0.24897 -0.23673 rpy=-1.3208 0.10472 3.1416 -> xyz=-0.044744 -0.00017 0.1337 rpy=-4.462392654 -0.10472 0
- joint L_ring_MCP_joint: origin xyz=-0.055098 -0.24897 -0.23909 rpy=-1.3208 0.05236 3.1416 -> xyz=-0.022902 -0.00017 0.13606 rpy=-4.462392654 -0.05236 0
- joint L_thumb_MCP_joint1: limit lower=0.3 upper=1.4 effort=50 velocity=1 -> lower=0 upper=1.1 effort=50 velocity=1; origin xyz=-0.098633 -0.23173 -0.15826 rpy=-1.5708 0 -0.16939 -> xyz=0.020633 0.01707 0.05523 rpy=-4.71238898 0 -2.672202654
- joint L_thumb_MCP_joint2: limit lower=1.5 upper=2 effort=50 velocity=1 -> lower=0 upper=0.5 effort=50 velocity=1; origin xyz=-0.0115 0.005 0 rpy=2.1656 -1.5708 0 -> xyz=-0.0115 0.005 0 rpy=0.82401 -1.5708 0

File: paquetes_simulacion/inspire_hands/inspire_hand_r/urdf/inspire_hand_r.urdf (robot description, URDF)
Before this commit: robot inspire_hand_r, 14 links, 13 joints
Links:
- removed link world
Joints:
- removed joint fixed
- joint R_index_MCP_joint: origin xyz=-0.094559 -0.24897 0.054025 rpy=1.3268 0.034907 3.1416 -> xyz=-0.016259 -0.00017 0.137085 rpy=1.3268 0.034907 3.1416
- joint R_middle_MCP_joint: origin xyz=-0.077068 -0.24897 0.054042 rpy=1.3208 0 3.1416 -> xyz=0.001232 -0.00017 0.137102 rpy=1.3208 0 3.1416
- joint R_pinky_MCP_joint: origin xyz=-0.038882 -0.24897 0.051205 rpy=1.3208 -0.10472 -3.1416 -> xyz=0.039418 -0.00017 0.134265 rpy=1.3208 -0.10472 -3.1416
- joint R_ring_MCP_joint: origin xyz=-0.057894 -0.24897 0.053119 rpy=1.3208 -0.05236 3.1416 -> xyz=0.020406 -0.00017 0.136179 rpy=1.3208 -0.05236 3.1416
- joint R_thumb_MCP_joint1: limit lower=0.2 upper=1.3 effort=50 velocity=1 -> lower=0 upper=1.1 effort=50 velocity=1; origin xyz=-0.098633 -0.23173 -0.011364 rpy=1.5708 0 -0.28289 -> xyz=-0.020333 0.01707 0.071696 rpy=1.5708 -0.2 -0.28289
- joint R_thumb_MCP_joint2: axis -1 0 0 -> 1 0 0; limit lower=1.3 upper=1.8 effort=50 velocity=1 -> lower=0 upper=0.5 effort=50 velocity=1; origin xyz=-0.0115 -0.011843 0 rpy=0.97599 1.5708 0 -> xyz=-0.0115 -0.011843 0 rpy=-0.82401 1.5708 0

File: paquetes_simulacion/rb1_base_description/robots/robot_wh.urdf (robot description, URDF)
Before this commit: robot rb1_base, 67 links, 66 joints
Links:
- removed link L_hand_base_link
- removed link L_index_distal
- removed link L_index_proximal
- removed link L_middle_distal
- removed link L_middle_proximal
- removed link L_pinky_distal
- removed link L_pinky_proximal
- removed link L_ring_distal
- removed link L_ring_proximal
- removed link L_thumb_distal
- removed link L_thumb_intermediate
- removed link L_thumb_proximal
- removed link L_thumb_proximal_base
- removed link R_hand_base_link
- removed link R_index_distal
- removed link R_index_proximal
- removed link R_middle_distal
- removed link R_middle_proximal
- removed link R_pinky_distal
- removed link R_pinky_proximal
- removed link R_ring_distal
- removed link R_ring_proximal
- removed link R_thumb_distal
- removed link R_thumb_intermediate
- removed link R_thumb_proximal
- removed link R_thumb_proximal_base
Joints:
- removed joint L_index_DIP_joint
- removed joint L_index_MCP_joint
- removed joint L_middle_DIP_joint
- removed joint L_middle_MCP_joint
- removed joint L_pinky_DIP_joint
- removed joint L_pinky_MCP_joint
- removed joint L_ring_DIP_joint
- removed joint L_ring_MCP_joint
- removed joint L_thumb_DIP_joint
- removed joint L_thumb_MCP_joint1
- removed joint L_thumb_MCP_joint2
- removed joint L_thumb_PIP_joint
- removed joint R_index_DIP_joint
- removed joint R_index_MCP_joint
- removed joint R_middle_DIP_joint
- removed joint R_middle_MCP_joint
- removed joint R_pinky_DIP_joint
- removed joint R_pinky_MCP_joint
- removed joint R_ring_DIP_joint
- removed joint R_ring_MCP_joint
- removed joint R_thumb_DIP_joint
- removed joint R_thumb_MCP_joint1
- removed joint R_thumb_MCP_joint2
- removed joint R_thumb_PIP_joint
- removed joint left_hand_base_joint
- removed joint right_hand_base_joint
